File: kicad_files/RP Uno.kicad_pcb (KiCad board)
At the start: 2 copper layers, 68.6 x 53.3 mm, 73 parts, among them J1 USB_B, J2 Conn_01x08, J3 Conn_01x06, J4 Conn_01x10, J5 Conn_01x08, J6 Barrel_Jack_Switch, J7 ICSP, J8 SWD, Q1 FDN340P, Q2 FDN340P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

Commit message: Partial Rev 2 updates
Parts:
- added D1: D_Schottky, Diode_SMD:D_SOD-323, F.Cu at (190.9, 97.9)
- J2, J5: value Conn_01x08 -> 8pin
- J3: value Conn_01x06 -> 6pin
- J4: value Conn_01x10 -> 10pin
- moved SW2 14.5 mm to (174.6, 93.7), turned to 0 degrees
- moved D1 10.9 mm to (171.4, 93.7), turned to -90 degrees
- moved R7 8.91 mm to (169.1, 94.5)
- moved R9 8.89 mm to (169.1, 93.0)
- moved U4 1.56 mm to (166.2, 98.6), turned to -45 degrees
Connections:
- D2 pad 1: Net-(D2-Pad1) -> /VIN
- R7 pad 2: Net-(D1-Pad2) -> Net-(R7-Pad2)
- SW2 pad 1: Net-(D1-Pad1) -> Net-(SW2-Pad1)
Routing:
- net +3V3: track 233.7 -> 194.7 mm, vias 19 -> 17
- net /QSPI_CS: track 32.0 -> 13.7 mm
- net /QSPI_DATA1: track 25.6 -> 12.2 mm
- net /QSPI_DATA3: track 9.26 -> 21.7 mm
- net /QSPI_DATA2: track 23.1 -> 10.8 mm
- net /QSPI_SCK: track 9.92 -> 20.1 mm
- net /QSPI_DATA0: track 10.6 -> 18.5 mm
- net Net-(D1-Pad1): track 1.93 -> 0.00 mm
- net Net-(D1-Pad2): track 1.49 -> 0.00 mm
